File: sr_circuit/sr_circuit.kicad_sch (KiCad schematic)
At the start: 11 parts, among them Q1 IRL540N, Q2 IRL540N, U1 ESP32-S3-DevKitC

Commit message: change names and resistor values
Parts:
- RG1, RG2: value 1K -> 100
- RGND1: renamed from RGND; value 1K -> 10K
- RGND2: renamed from RGND1; value 1K -> 10K
Changed lines of the file:
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@@
 			)
 		)
-		(property "Value" "1K"
+		(property "Value" "100"
 			(at 128.27 121.92 0)
 			(effects
@@
 		(on_board yes)
 		(dnp no)
-		(property "Reference" "RGND"
+		(property "Reference" "RGND1"
 			(at 131.318 85.09 0)
 			(effects
@@
 			)
 		)
-		(property "Value" "1K"
+		(property "Value" "10K"
 			(at 130.81 85.09 0)
 			(effects
@@
 			(project "sr_circuit"
 				(path "/cfda6094-67cc-46d2-af38-a5b6e7551bb5"
-					(reference "RGND")
+					(reference "RGND1")
 					(unit 1)
 				)
@@
 			)
 		)
-		(property "Value" "1K"
+		(property "Value" "100"
 			(at 127 74.93 0)
 			(effects
@@
 		(on_board yes)
 		(dnp no)
-		(property "Reference" "RGND1"
+		(property "Reference" "RGND2"
 			(at 132.588 132.08 0)
 			(effects
@@
 			)
 		)
-		(property "Value" "1K"
+		(property "Value" "10K"
 			(at 132.08 132.08 0)
 			(effects
@@
 			(project "sr_circuit"
 				(path "/cfda6094-67cc-46d2-af38-a5b6e7551bb5"
-					(reference "RGND1")
-					(unit 1)
-				)
+					(reference "RGND2")
+					(unit 1)
+				)

Commit message: add external power supply
Parts:
- added J1: Barrel_Jack, Connector_BarrelJack:BarrelJack_SwitchcraftConxall_RAPC10U_Horizontal, symbol Connector:Barrel_Jack
- added U2: L7805, PCM_Package_TO_SOT_SMD_AKL:TO-252-2, symbol Regulator_Linear:L7805
Connections:
- net +12V: now also J1.1, U2.1 (IN)
- net GND: now also J1.2, U2.2 (GND)
- net 5VPS: now reaches U1.21 (5V)
- net 5VPS: now also U2.3 (OUT)
- no-connect marks 33 -> 32

Commit message: add buckboost IC
Parts:
- removed U2: L7805, PCM_Package_TO_SOT_SMD_AKL:TO-252-2, symbol Regulator_Linear:L7805
- added U2: LM2596S-3.3, Package_TO_SOT_SMD:TO-263-5_TabPin3, symbol Regulator_Switching:LM2596S-3.3
Connections:
- net +12V: now also U2.1 (VIN)
- net 3V3: now also U2.2 (OUT)
- net GND: now also U2.3 (GND), U2.5 (~{ON}/OFF)
- no-connect marks 32 -> 34
Other:
- moved on the sheet: J1
